File: receiver.sch (EAGLE design)
At the start: 33 parts

Commit message: Changed labels.
Parts:
- removed B1: DTS-3, switch-tact:DTS-3
- added S5: SWS001, smd-special:SWS001
- S1: value SWS001 -> DTS-6; device smd-special:SWS001 -> switch-tact:DTS-6
- renumbered SV1 to OLED
Connections:
- removed net N$1: B1.2, R1.1, R2.1
- new net N$14: R1.1, R2.1, S1.3, S1.4
- net GND: now also S1.2, S5.1; no longer B1.1
- net N$3: now also S5.2; no longer S1.2
Changed lines of the file:
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@@
 <part name="GND8" library="supply1" library_urn="urn:adsk.eagle:library:371" deviceset="GND" device=""/>
 <part name="R13" library="rcl" library_urn="urn:adsk.eagle:library:334" deviceset="R-EU_" device="0204/5" package3d_urn="urn:adsk.eagle:package:23488/1" value="2k2"/>
-<part name="S1" library="smd-special" library_urn="urn:adsk.eagle:library:362" deviceset="SWS001" device="" package3d_urn="urn:adsk.eagle:package:26467/1"/>
+<part name="S5" library="smd-special" library_urn="urn:adsk.eagle:library:362" deviceset="SWS001" device="" package3d_urn="urn:adsk.eagle:package:26467/1"/>
 <part name="GND2" library="supply1" library_urn="urn:adsk.eagle:library:371" deviceset="GND" device=""/>
 <part name="GND10" library="supply1" library_urn="urn:adsk.eagle:library:371" deviceset="GND" device=""/>
@@
 <part name="SUPPLY13" library="supply2" library_urn="urn:adsk.eagle:library:372" deviceset="VCC" device="" value="+3V3"/>
 <part name="SUPPLY14" library="supply2" library_urn="urn:adsk.eagle:library:372" deviceset="VCC" device="" value="+3V3"/>
-<part name="B1" library="switch-tact" deviceset="DTS-3" device=""/>
 <part name="R1" library="rcl" library_urn="urn:adsk.eagle:library:334" deviceset="R-EU_" device="0204/5" package3d_urn="urn:adsk.eagle:package:23488/1" value="10k"/>
 <part name="GND9" library="supply1" library_urn="urn:adsk.eagle:library:371" deviceset="GND" device=""/>
@@
 <part name="S3" library="switch-tact" deviceset="DTS-6" device=""/>
 <part name="S4" library="switch-tact" deviceset="DTS-6" device=""/>
-<part name="SV1" library="con-lsta" library_urn="urn:adsk.eagle:library:161" deviceset="FE08-1" device="" package3d_urn="urn:adsk.eagle:package:8194/1"/>
+<part name="OLED" library="con-lsta" library_urn="urn:adsk.eagle:library:161" deviceset="FE08-1" device="" package3d_urn="urn:adsk.eagle:package:8194/1"/>
 <part name="R17" library="rcl" library_urn="urn:adsk.eagle:library:334" deviceset="R-EU_" device="0204/5" package3d_urn="urn:adsk.eagle:package:23488/1" value="4,7k"/>
 <part name="SUPPLY15" library="supply2" library_urn="urn:adsk.eagle:library:372" deviceset="VCC" device="" value="+3V3"/>
+<part name="S1" library="switch-tact" deviceset="DTS-6" device=""/>
 </parts>
 <sheets>
@@
 <instance part="GND8" gate="1" x="10.16" y="101.6"/>
 <instance part="R13" gate="G$1" x="101.6" y="58.42"/>
-<instance part="S1" gate="G$1" x="109.22" y="50.8" rot="R90"/>
+<instance part="S5" gate="G$1" x="109.22" y="50.8" rot="R90"/>
 <instance part="GND2" gate="1" x="119.38" y="45.72"/>
 <instance part="GND10" gate="1" x="27.94" y="27.94"/>
@@
 <instance part="SUPPLY13" gate="G$1" x="12.7" y="53.34"/>
 <instance part="SUPPLY14" gate="G$1" x="40.64" y="50.8"/>
-<instance part="B1" gate="G$1" x="20.32" y="78.74" rot="R270"/>
 <instance part="R1" gate="G$1" x="25.4" y="91.44" rot="R90"/>
-<instance part="GND9" gate="1" x="10.16" y="73.66"/>
+<instance part="GND9" gate="1" x="0" y="73.66"/>
 <instance part="R15" gate="G$1" x="129.54" y="60.96" rot="R90"/>
 <instance part="R16" gate="G$1" x="134.62" y="81.28" rot="R90"/>
@@
 <instance part="S3" gate="G$1" x="7.62" y="43.18"/>
 <instance part="S4" gate="G$1" x="25.4" y="40.64"/>
-<instance part="SV1" gate="G$1" x="170.18" y="73.66" rot="R180"/>
+<instance part="OLED" gate="G$1" x="170.18" y="73.66" rot="R180"/>
 <instance part="R17" gate="G$1" x="157.48" y="55.88" rot="R90"/>
 <instance part="SUPPLY15" gate="G$1" x="165.1" y="50.8"/>
+<instance part="S1" gate="G$1" x="12.7" y="81.28" rot="R270"/>
 </instances>
 <busses>
@@
 </segment>
 <segment>
-<pinref part="S1" gate="G$1" pin="1"/>
+<pinref part="S5" gate="G$1" pin="1"/>
 <wire x1="114.3" y1="50.8" x2="119.38" y2="50.8" width="0.1524" layer="91"/>
 <wire x1="119.38" y1="50.8" x2="119.38" y2="48.26" width="0.1524" layer="91"/>
@@
 </segment>
 <segment>
-<pinref part="B1" gate="G$1" pin="1"/>
-<wire x1="15.24" y1="78.74" x2="10.16" y2="78.74" width="0.1524" layer="91"/>
-<pinref part="GND9" gate="1" pin="GND"/>
-<wire x1="10.16" y1="78.74" x2="10.16" y2="76.2" width="0.1524" layer="91"/>
-</segment>
-<segment>
 <pinref part="GND7" gate="1" pin="GND"/>
 <wire x1="-10.16" y1="40.64" x2="-10.16" y2="38.1" width="0.1524" layer="91"/>
@@
 </segment>
 <segment>
-<pinref part="SV1" gate="G$1" pin="2"/>
+<pinref part="OLED" gate="G$1" pin="2"/>
 <wire x1="162.56" y1="78.74" x2="152.4" y2="78.74" width="0.1524" layer="91"/>
 <wire x1="152.4" y1="78.74" x2="152.4" y2="88.9" width="0.1524" layer="91"/>
@@
 <wire x1="144.78" y1="88.9" x2="144.78" y2="86.36" width="0.1524" layer="91"/>
 </segment>
-</net>
-<net name="N$1" class="0">
-<segment>
-<pinref part="R1" gate="G$1" pin="1"/>
-<pinref part="B1" gate="G$1" pin="2"/>
-<wire x1="25.4" y1="86.36" x2="25.4" y2="78.74" width="0.1524" layer="91"/>
-<pinref part="R2" gate="G$1" pin="1"/>
-<wire x1="27.94" y1="78.74" x2="25.4" y2="78.74" width="0.1524" layer="91"/>
-<junction x="25.4" y="78.74"/>
+<segment>
+<pinref part="S1" gate="G$1" pin="2"/>
+<wire x1="7.62" y1="78.74" x2="5.08" y2="78.74" width="0.1524" layer="91"/>
+<pinref part="GND9" gate="1" pin="GND"/>
+<wire x1="5.08" y1="78.74" x2="0" y2="78.74" width="0.1524" layer="91"/>
+<wire x1="0" y1="78.74" x2="0" y2="76.2" width="0.1524" layer="91"/>
+<pinref part="S1" gate="G$1" pin="1"/>
+<wire x1="7.62" y1="81.28" x2="5.08" y2="81.28" width="0.1524" layer="91"/>
+<wire x1="5.08" y1="81.28" x2="5.08" y2="78.74" width="0.1524" layer="91"/>
+<junction x="5.08" y="78.74"/>
 </segment>
 </net>
@@
 <wire x1="129.54" y1="68.58" x2="149.86" y2="68.58" width="0.1524" layer="91"/>
 <wire x1="149.86" y1="68.58" x2="149.86" y2="71.12" width="0.1524" layer="91"/>
-<pinref part="SV1" gate="G$1" pin="5"/>
+<pinref part="OLED" gate="G$1" pin="5"/>
 <wire x1="149.86" y1="71.12" x2="162.56" y2="71.12" width="0.1524" layer="91"/>
 </segment>
@@
 <wire x1="162.56" y1="73.66" x2="134.62" y2="73.66" width="0.1524" layer="91"/>
 <junction x="134.62" y="73.66"/>
-<pinref part="SV1" gate="G$1" pin="4"/>
+<pinref part="OLED" gate="G$1" pin="4"/>
 </segment>
 </net>
@@
 <wire x1="91.44" y1="58.42" x2="91.44" y2="50.8" width="0.1524" layer="91"/>
 <wire x1="91.44" y1="50.8" x2="101.6" y2="50.8" width="0.1524" layer="91"/>
-<pinref part="S1" gate="G$1" pin="2"/>
+<pinref part="S5" gate="G$1" pin="2"/>
 <pinref part="R14" gate="G$1" pin="2"/>
 <wire x1="88.9" y1="63.5" x2="91.44" y2="63.5" width="0.1524" layer="91"/>
@@
 <net name="N$8" class="0">
 <segment>
-<pinref part="SV1" gate="G$1" pin="8"/>
+<pinref part="OLED" gate="G$1" pin="8"/>
 <wire x1="162.56" y1="63.5" x2="157.48" y2="63.5" width="0.1524" layer="91"/>
 <wire x1="157.48" y1="63.5" x2="157.48" y2="60.96" width="0.1524" layer="91"/>
 </segment>
 </net>
+<net name="N$14" class="0">
+<segment>
+<pinref part="S1" gate="G$1" pin="3"/>
+<wire x1="17.78" y1="81.28" x2="20.32" y2="81.28" width="0.1524" layer="91"/>
+<wire x1="20.32" y1="81.28" x2="20.32" y2="78.74" width="0.1524" layer="91"/>
+<pinref part="S1" gate="G$1" pin="4"/>
+<wire x1="20.32" y1="78.74" x2="17.78" y2="78.74" width="0.1524" layer="91"/>
+<pinref part="R1" gate="G$1" pin="1"/>
+<wire x1="25.4" y1="86.36" x2="25.4" y2="78.74" width="0.1524" layer="91"/>
+<pinref part="R2" gate="G$1" pin="1"/>
+<wire x1="27.94" y1="78.74" x2="25.4" y2="78.74" width="0.1524" layer="91"/>
+<wire x1="20.32" y1="78.74" x2="25.4" y2="78.74" width="0.1524" layer="91"/>
+<junction x="20.32" y="78.74"/>
+<junction x="25.4" y="78.74"/>
+</segment>
+</net>

Commit message: Changed +3V7 for V_BAT and deleted some errors.
Connections:
- net N$8: now also R17.2
- net VCC: now also OLED.1
Changed lines of the file:
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@@
 <part name="LI-POL" library="pinhead" library_urn="urn:adsk.eagle:library:325" deviceset="PINHD-1X2" device="" package3d_urn="urn:adsk.eagle:package:22435/2"/>
 <part name="GND6" library="supply1" library_urn="urn:adsk.eagle:library:371" deviceset="GND" device=""/>
-<part name="SUPPLY9" library="supply2" library_urn="urn:adsk.eagle:library:372" deviceset="VCC" device="" value="+3V7"/>
+<part name="SUPPLY9" library="supply2" library_urn="urn:adsk.eagle:library:372" deviceset="VCC" device="" value="V_BAT"/>
 <part name="R10" library="rcl" library_urn="urn:adsk.eagle:library:334" deviceset="R-EU_" device="0204/5" package3d_urn="urn:adsk.eagle:package:23488/1" value="100"/>
 <part name="C1" library="rcl" library_urn="urn:adsk.eagle:library:334" deviceset="CPOL-EU" device="E2.5-6" package3d_urn="urn:adsk.eagle:package:23349/1" value="100u"/>
 <part name="C2" library="rcl" library_urn="urn:adsk.eagle:library:334" deviceset="C-EU" device="025-025X050" package3d_urn="urn:adsk.eagle:package:23629/2" value="100n"/>
-<part name="SUPPLY3" library="supply2" library_urn="urn:adsk.eagle:library:372" deviceset="VCC" device="" value="+3V7"/>
+<part name="SUPPLY3" library="supply2" library_urn="urn:adsk.eagle:library:372" deviceset="VCC" device="" value="V_BAT"/>
 <part name="GND8" library="supply1" library_urn="urn:adsk.eagle:library:371" deviceset="GND" device=""/>
 <part name="R13" library="rcl" library_urn="urn:adsk.eagle:library:334" deviceset="R-EU_" device="0204/5" package3d_urn="urn:adsk.eagle:package:23488/1" value="2k2"/>
@@
 </segment>
 <segment>
-<wire x1="162.56" y1="81.28" x2="154.94" y2="81.28" width="0.1524" layer="91"/>
 <wire x1="154.94" y1="81.28" x2="154.94" y2="86.36" width="0.1524" layer="91"/>
 <pinref part="SUPPLY7" gate="G$1" pin="VCC"/>
+<pinref part="OLED" gate="G$1" pin="1"/>
+<wire x1="154.94" y1="81.28" x2="162.56" y2="81.28" width="0.1524" layer="91"/>
 </segment>
 <segment>
@@
 <wire x1="10.16" y1="106.68" x2="10.16" y2="104.14" width="0.1524" layer="91"/>
 <pinref part="GND8" gate="1" pin="GND"/>
+<junction x="10.16" y="106.68"/>
 </segment>
 <segment>
@@
 <pinref part="OLED" gate="G$1" pin="8"/>
 <wire x1="162.56" y1="63.5" x2="157.48" y2="63.5" width="0.1524" layer="91"/>
-<wire x1="157.48" y1="63.5" x2="157.48" y2="60.96" width="0.1524" layer="91"/>
-</segment>
-</net>
+<pinref part="R17" gate="G$1" pin="2"/>
+<wire x1="157.48" y1="60.96" x2="157.48" y2="63.5" width="0.1524" layer="91"/>
+</segment>
+</net>

Commit message: Boards and schematics are done.
Parts:
- removed SU/SD3V3: 5V_VOLTAGE_REGULATOR, Pololu Voltage Regulators:5V_VOLTAGE_REGULATOR
- added SD: (no value), pinhead:PINHD-1X4
- R1, R10, R11, R12, R13, R14, R15, R16, R17, R2, R3, R4, R5, R6, R7, R8, R9: device rcl:R-EU_0204/5 -> rcl:R-EU_0204/7
- S5: value SWS001 -> -SWITCH; device smd-special:SWS001 -> tango:-SWITCH
Connections:
- new net V+: C1.+, C2.1, C3.1, SD.2, U$1.OUT+
- net GND: now also S5.2, SD.3; no longer S5.1, SU/SD3V3.GND
- net N$3: now also S5.1; no longer S5.2
- net VCC: now also SD.4; no longer C1.+, C2.1, C3.1, SU/SD3V3.VIN, SU/SD3V3.VOUT, U$1.OUT+
Other:
- moved on the sheet: C3, C4
